File: wired-sculpt.kicad_pcb (KiCad board)
At the start: 2 copper layers, 40 x 50 mm, 39 parts, among them J1 10103594-0001LF, J2 FFC3B07-30-T, J3 AVR-ISP-6 - NOT FITTED, Q1 BSS84AK,215, Q2 2N7002BK, SW1 FSMSM, SW2 S2B-PH-K-S(LF)(SN), U1 USBLC6-2SC6, U2 LM2776DBVT, U3 AT90USB1286-AU, Y1 TSX-3225 16.0000MF18X-AC0

Commit message: Update Kicad files to Kicad 6.0
Other:
- net class Default removed
- net class Fat removed
